File: pcb/strato_connect.kicad_pcb (KiCad board)
At the start: 4 copper layers, 38.6 x 40.3 mm, 49 parts, among them J1 Conn_Coaxial, J2 Conn_01x04_Pin, J3 Conn_01x04_Pin, J5 Conn_01x01_Pin, J6 Conn_01x02_Pin, SW1 SW_SPST, U1 TPS565242, U2 ATmega328PB-M, U4 RF4463F30, Y1 CSTNE16M0V530000R0

Commit message: add v2 files for the pcb, add the base code directory
Parts:
- C7: value 47u -> 100u
Changed lines of the file:
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@@
     (property "ki_description" "Unpolarized capacitor")
     (property "ki_keywords" "cap capacitor")
-    (attr smd)
+    (attr smd exclude_from_bom)
     (fp_text reference "C9" (at 0 -1.16 90) (layer "F.SilkS") hide
         (effects (font (size 1 1) (thickness 0.15)))
@@
         (effects (font (size 1 1) (thickness 0.15)))
     )
-    (fp_text value "47u" (at 0 3.7) (layer "F.Fab") hide
+    (fp_text value "100u" (at 0 3.7) (layer "F.Fab") hide
         (effects (font (size 1 1) (thickness 0.15)))
     )
@@
     (property "ki_description" "Resistor, small US symbol")
     (property "ki_keywords" "r resistor")
-    (attr smd)
-    (fp_text reference "R12" (at 0 -1.17 -90) (layer "F.SilkS") hide
-        (effects (font (size 1 1) (thickness 0.15)))
-    )
-    (fp_text value "NP" (at 0 1.17 -90) (layer "F.Fab") hide
-        (effects (font (size 1 1) (thickness 0.15)))
-    )
-    (fp_text user "${REFERENCE}" (at 0 0 -90) (layer "F.Fab")
+    (attr smd exclude_from_bom)
+    (fp_text reference "R12" (at 0 -1.17 90) (layer "F.SilkS") hide
+        (effects (font (size 1 1) (thickness 0.15)))
+    )
+    (fp_text value "NP" (at 0 1.17 90) (layer "F.Fab") hide
+        (effects (font (size 1 1) (thickness 0.15)))
+    )
+    (fp_text user "${REFERENCE}" (at 0 0 90) (layer "F.Fab")
         (effects (font (size 0.26 0.26) (thickness 0.04)))
     )

Commit message: update programming pcb so it can be secured to the stemma grid
Other:
- board text added: "delta x between h3 pin 1 of the programming header: 6.68900 mm 0.26334 inch"
Changed lines of the file:
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@@
   (gr_line (start 170.8 57.7) (end 171 57.7)
     (stroke (width 0.1) (type default)) (layer "Edge.Cuts"))
+  (gr_text "delta x between h3 pin 1 of \nthe programming header:\n6.68900 mm\n0.26334 inch" (at 114.7318 75.7174) (layer "Cmts.User")
+    (effects (font (size 1.5 1.5) (thickness 0.3) bold) (justify left bottom))
+  )
   (gr_text "For colplanar:\n0.777mm trace width\n0.15mm spacing" (at 180.3 66.9) (layer "Cmts.User")
     (effects (font (size 1.5 1.5) (thickness 0.3) bold) (justify left bottom))
